File: pcb/audio.sch (KiCad schematic (older format))
At the start: 12 parts, among them U3 PAM8403DR

Commit message: First submitted PCB
Parts:
- U3: footprint SOIC127P605X150-16N -> lib:SOIC127P605X150-16N
Connections:
- net GND: now also C15.1, C16.1, C17.1, C18.2
Changed lines of the file:
@@
 LIBS:PAM8403DR
 LIBS:JQ1P-5V-F
+LIBS:Connector_Generic_MountingPin
 LIBS:controller-cache
 EELAYER 25 0
@@
 F 0 "U3" H 5199 3971 50  0000 L BNN
 F 1 "PAM8403DR" H 5199 2348 50  0000 L BNN
-F 2 "SOIC127P605X150-16N" H 5600 3250 50  0001 L BNN
+F 2 "lib:SOIC127P605X150-16N" H 5600 3250 50  0001 L BNN
 F 3 "Diodes" H 5600 3250 50  0001 L BNN
 F 4 "Diodes Inc" H 5600 3250 60  0001 C CNN "Manufacturer"
@@
 	6200 2850 6200 2450
 $Comp
-L +3V3 #PWR017
+L +3V3 #PWR015
 U 1 1 5F392BFE
 P 6200 2450
-F 0 "#PWR017" H 6200 2300 50  0001 C CNN
+F 0 "#PWR015" H 6200 2300 50  0001 C CNN
 F 1 "+3V3" H 6200 2590 50  0000 C CNN
 F 2 "" H 6200 2450 50  0001 C CNN
@@
 $EndComp
 $Comp
-L GND #PWR018
+L GND #PWR016
 U 1 1 5F392CC4
 P 6200 4200
-F 0 "#PWR018" H 6200 3950 50  0001 C CNN
+F 0 "#PWR016" H 6200 3950 50  0001 C CNN
 F 1 "GND" H 6200 4050 50  0000 C CNN
 F 2 "" H 6200 4200 50  0001 C CNN
@@
 Connection ~ 6800 2800
 $Comp
-L GND #PWR019
+L GND #PWR017
 U 1 1 5F3931E7
 P 6900 2800
-F 0 "#PWR019" H 6900 2550 50  0001 C CNN
+F 0 "#PWR017" H 6900 2550 50  0001 C CNN
 F 1 "GND" H 6900 2650 50  0000 C CNN
 F 2 "" H 6900 2800 50  0001 C CNN
@@
 	3350 3200 3350 3300
 $Comp
-L GND #PWR020
+L GND #PWR018
 U 1 1 5F397B0B
 P 3400 3250
-F 0 "#PWR020" H 3400 3000 50  0001 C CNN
+F 0 "#PWR018" H 3400 3000 50  0001 C CNN
 F 1 "GND" H 3400 3100 50  0000 C CNN
 F 2 "" H 3400 3250 50  0001 C CNN
@@
 Connection ~ 6200 3750
 Connection ~ 6200 4200
+Connection ~ 6900 2800
 $EndSCHEMATC

Commit message: Fixes after board arrived
Parts:
- C12, C13: value C -> 470nf
Changed lines of the file:
@@
 LIBS:PAM8403DR
 LIBS:JQ1P-5V-F
-LIBS:Connector_Generic_MountingPin
 LIBS:controller-cache
 EELAYER 25 0
@@
 P 4300 3050
 F 0 "C12" H 4325 3150 50  0000 L CNN
-F 1 "C" H 4325 2950 50  0000 L CNN
+F 1 "470nf" H 4325 2950 50  0000 L CNN
 F 2 "Capacitors_SMD:C_0603_HandSoldering" H 4338 2900 50  0001 C CNN
 F 3 "" H 4300 3050 50  0001 C CNN
@@
 P 4300 3250
 F 0 "C13" H 4325 3350 50  0000 L CNN
-F 1 "C" H 4325 3150 50  0000 L CNN
+F 1 "470nf" H 4325 3150 50  0000 L CNN
 F 2 "Capacitors_SMD:C_0603_HandSoldering" H 4338 3100 50  0001 C CNN
 F 3 "" H 4300 3250 50  0001 C CNN
