File: pcb/external.sch (KiCad schematic (older format))
At the start: 40 parts, among them J1 Steering, J10 SPK_L_OUT, J11 Batt, J12 Motor, J2 Volume, J3 Light, J4 Gas_In, J5 Direction, J6 Light_Out, J7 LED_Out, J8 uSD, J9 SPK_R_OUT

Commit message: First submitted PCB
Parts:
- added J13: ACC, Connectors_JST:JST_XH_B02B-XH-A_02x2.50mm_Straight, symbol Conn_01x02
- added K3: JQ1P-5V-F, lib:JQ1P5VF, symbol JQ1P-5V-F
- added M1, M2, M3, M4: M3, Mounting_Holes:MountingHole_3.2mm_M3_Pad, symbol Screw_Terminal_01x01
- J10, J3, J4, J6, J7, J9: footprint (none) -> Connectors_JST:JST_XH_B02B-XH-A_02x2.50mm_Straight
- J11, J12: footprint (none) -> Connectors_JST:JST_VH_B2P-VH-B_2x3.96mm_Vertical
Connections:
- net +BATT: now also K3.1 (COIL_1), K3.4 (COM)
- net GND: now also J13.2 (Pin_2), M1.1 (Pin_1), M2.1 (Pin_1), M3.1 (Pin_1), M4.1 (Pin_1)
- new net: J13.1 (Pin_1), K3.5 (COIL_2)
- new net ACC_BAT: K3.3 (NO)
- no-connect marks 0 -> 1
