File: pcb/mcu.sch (KiCad schematic (older format))
At the start: 17 parts, among them U1 ULN2803A, U2 STM32F405RGTx

Commit message: First submitted PCB
Parts:
- JP1: footprint 20021221-00010C4LF -> lib:20021221-00010C4LF
- U2: footprint LQFP64 -> Housings_QFP:LQFP-64_10x10mm_Pitch0.5mm
Connections:
- net +3V3: now also C1.1, C2.1, C3.1, C4.1, C5.1, C6.1, C7.1
- net BWD_IN: now also U2.33 (PB12/CAN2_RX/I2C2_SMBA/I2S2_WS/SPI2_NSS/TIM1_BKIN/USART3_CK/USB_OTG_HS_ID/USB_OTG_HS_ULPI_D5); no longer U2.34 (PB13/CAN2_TX/I2S2_CK/SPI2_SCK/TIM1_CH1N/USART3_CTS/USB_OTG_HS_ULPI_D6/USB_OTG_HS_VBUS)
- net FWD_IN: now also U2.34 (PB13/CAN2_TX/I2S2_CK/SPI2_SCK/TIM1_CH1N/USART3_CTS/USB_OTG_HS_ULPI_D6/USB_OTG_HS_VBUS); no longer U2.33 (PB12/CAN2_RX/I2C2_SMBA/I2S2_WS/SPI2_NSS/TIM1_BKIN/USART3_CK/USB_OTG_HS_ID/USB_OTG_HS_ULPI_D5)
- net GND: now also C1.2, C2.2, C3.2, C4.2, C5.2, C6.2, C7.2
- net LAMP_OUT_SIG: now also U2.8 (PC0/ADC1_IN10/ADC2_IN10/ADC3_IN10/USB_OTG_HS_ULPI_STP); no longer U2.11 (PC3/ADC1_IN13/ADC2_IN13/ADC3_IN13/I2S2_SD/SPI2_MOSI/USB_OTG_HS_ULPI_NXT)
- net LED_OUT_SIG: now also U2.9 (PC1/ADC1_IN11/ADC2_IN11/ADC3_IN11); no longer U2.10 (PC2/ADC1_IN12/ADC2_IN12/ADC3_IN12/I2S2_ext_SD/SPI2_MISO/USB_OTG_HS_ULPI_DIR)
- net MOTOR_1_OUT_SIG: now also U2.11 (PC3/ADC1_IN13/ADC2_IN13/ADC3_IN13/I2S2_SD/SPI2_MOSI/USB_OTG_HS_ULPI_NXT); no longer U2.8 (PC0/ADC1_IN10/ADC2_IN10/ADC3_IN10/USB_OTG_HS_ULPI_STP)
- net MOTOR_2_OUT_SIG: now also U2.10 (PC2/ADC1_IN12/ADC2_IN12/ADC3_IN12/I2S2_ext_SD/SPI2_MISO/USB_OTG_HS_ULPI_DIR); no longer U2.9 (PC1/ADC1_IN11/ADC2_IN11/ADC3_IN11)
Changed lines of the file:
@@
 LIBS:PAM8403DR
 LIBS:JQ1P-5V-F
+LIBS:Connector_Generic_MountingPin
 LIBS:controller-cache
 EELAYER 25 0
@@
 F 0 "U2" H 8150 5000 50  0000 C CNN
 F 1 "STM32F405RGTx" H 8150 4800 50  0000 C CNN
-F 2 "LQFP64" H 8150 4700 50  0000 C CIN
+F 2 "Housings_QFP:LQFP-64_10x10mm_Pitch0.5mm" H 8150 4700 50  0000 C CIN
 F 3 "" H 8150 4900 50  0000 C CNN
 F 4 "STM32F405RGT6" H 8150 4900 60  0001 C CNN "MFRPN"
@@
 Text HLabel 14150 4400 2    60   Input ~ 0
 SD_CMD
+Text HLabel 14150 4000 2    60   Input ~ 0
+FWD_IN
 Text HLabel 14150 3900 2    60   Input ~ 0
-FWD_IN
-Text HLabel 14150 4000 2    60   Input ~ 0
 BWD_IN
 Text HLabel 14150 4100 2    60   Input ~ 0
@@
 F 0 "JP1" H 1600 10325 50  0000 L BNN
 F 1 "20021221-00010C4LF" H 1600 9599 50  0000 L BNN
-F 2 "20021221-00010C4LF" H 1850 10000 50  0001 L BNN
+F 2 "lib:20021221-00010C4LF" H 1850 10000 50  0001 L BNN
 F 3 "" H 1850 10000 60  0001 C CNN
 	1    1850 10000
@@
 	1    0    0    -1
 $EndComp
-Wire Wire Line
-	1200 8650 3150 8650
-Connection ~ 1500 8650
 Connection ~ 1800 8650
 Connection ~ 2100 8650
 Connection ~ 2400 8650
-Wire Wire Line
-	1200 8950 3150 8950
-Connection ~ 1500 8950
 Connection ~ 1800 8950
 Connection ~ 2100 8950
@@
 F 3 "" H 1950 8950 50  0001 C CNN
 	1    1950 8950
-	1    0    0    -1
-$EndComp
-$Comp
-L C C2
-U 1 1 5F38A35E
-P 1500 8800
-F 0 "C2" H 1525 8900 50  0000 L CNN
-F 1 "100nF" H 1525 8700 50  0000 L CNN
-F 2 "Capacitors_SMD:C_0603_HandSoldering" H 1538 8650 50  0001 C CNN
-F 3 "" H 1500 8800 50  0001 C CNN
-F 4 "C184760" H 1500 8800 60  0001 C CNN "LCSC"
-F 5 "GCM188R71C104KA37D" H 1500 8800 60  0001 C CNN "MFRPN"
-F 6 "Murata" H 1500 8800 60  0001 C CNN "Manufacturer"
-	1    1500 8800
 	1    0    0    -1
 $EndComp
@@
 	13650 6400 14500 6400
 Wire Wire Line
-	13650 6500 14500 6500
-Wire Wire Line
 	14500 6500 14500 6650
 $Comp
@@
 Wire Wire Line
 	2650 4600 2000 4600
-Wire Wire Line
-	2650 4700 2000 4700
 Text HLabel 6550 9100 2    60   Output ~ 0
 MOTOR1_CTL
@@
 Wire Wire Line
 	6550 9400 6200 9400
-Text Label 2000 4700 0    60   ~ 0
+Text Label 2000 4400 0    60   ~ 0
 LAMP_OUT_SIG
 Wire Wire Line
@@
 Wire Wire Line
 	6200 9300 6550 9300
+Text Label 2000 4500 0    60   ~ 0
+LED_OUT_SIG
+Wire Wire Line
+	6550 9200 6200 9200
 Text Label 2000 4600 0    60   ~ 0
-LED_OUT_SIG
-Wire Wire Line
-	6550 9200 6200 9200
-Text Label 2000 4500 0    60   ~ 0
 MOTOR_2_OUT_SIG
 Text Label 4550 9200 0    60   ~ 0
@@
 Text Label 4550 9100 0    60   ~ 0
 MOTOR_1_OUT_SIG
-Text Label 2000 4400 0    60   ~ 0
+Text Label 2000 4700 0    60   ~ 0
 MOTOR_1_OUT_SIG
 Wire Wire Line
@@
 	0    1    1    0
 $EndComp
-Wire Wire Line
-	6300 9900 6200 9900
 $Comp
 L GND #PWR014
@@
 	0    1    1    0
 $EndComp
-Wire Wire Line
-	6300 10150 6300 9900
 Wire Wire Line
 	6000 10150 5800 10150
@@
 NoConn ~ 2050 10100
 Connection ~ 14900 6500
-$Comp
-L PWR_FLAG #FLG015
-U 1 1 5F3D56F7
-P 14200 6500
-F 0 "#FLG015" H 14200 6575 50  0001 C CNN
-F 1 "PWR_FLAG" H 14200 6650 50  0000 C CNN
-F 2 "" H 14200 6500 50  0001 C CNN
-F 3 "" H 14200 6500 50  0001 C CNN
-	1    14200 6500
-	-1   0    0    1
-$EndComp
-Connection ~ 14200 6500
-$Comp
-L PWR_FLAG #FLG016
-U 1 1 5F3D573E
-P 14500 6150
-F 0 "#FLG016" H 14500 6225 50  0001 C CNN
-F 1 "PWR_FLAG" H 14500 6300 50  0000 C CNN
-F 2 "" H 14500 6150 50  0001 C CNN
-F 3 "" H 14500 6150 50  0001 C CNN
-	1    14500 6150
-	1    0    0    -1
-$EndComp
-Wire Wire Line
-	14500 6400 14500 6150
-Connection ~ 14500 6400
+Connection ~ 13650 6700
+Wire Wire Line
+	13650 6500 14500 6500
+Connection ~ 6300 9900
+Wire Wire Line
+	6300 9900 6200 9900
+Wire Wire Line
+	6300 10150 6300 9900
+Connection ~ 1950 8950
+Connection ~ 1950 8650
+Connection ~ 1500 8950
+Connection ~ 1500 8650
+Wire Wire Line
+	1200 8650 3150 8650
+Wire Wire Line
+	1200 8950 3150 8950
+Wire Wire Line
+	2650 4700 2000 4700
+$Comp
+L C C2
+U 1 1 5F3E16E7
+P 1500 8800
+F 0 "C2" H 1525 8900 50  0000 L CNN
+F 1 "100nF" H 1525 8700 50  0000 L CNN
+F 2 "Capacitors_SMD:C_0603_HandSoldering" H 1538 8650 50  0001 C CNN
+F 3 "" H 1500 8800 50  0001 C CNN
+F 4 "C184760" H 1500 8800 60  0001 C CNN "LCSC"
+F 5 "GCM188R71C104KA37D" H 1500 8800 60  0001 C CNN "MFRPN"
+F 6 "Murata" H 1500 8800 60  0001 C CNN "Manufacturer"
+	1    1500 8800
+	1    0    0    -1
+$EndComp
 $EndSCHEMATC
