File: pcb/motor.sch (KiCad schematic (older format))
At the start: 2 parts, among them K1 JQ1P-5V-F, K2 JQ1P-5V-F

Commit message: First submitted PCB
Parts:
- K1: footprint JQ1P5VF -> lib:JQ1P5VF
Changed lines of the file:
@@
 LIBS:PAM8403DR
 LIBS:JQ1P-5V-F
+LIBS:Connector_Generic_MountingPin
 LIBS:controller-cache
 EELAYER 25 0
@@
 $EndComp
 $Comp
-L GND #PWR021
+L GND #PWR019
 U 1 1 5F3C9467
 P 2300 3700
-F 0 "#PWR021" H 2300 3450 50  0001 C CNN
+F 0 "#PWR019" H 2300 3450 50  0001 C CNN
 F 1 "GND" H 2300 3550 50  0000 C CNN
 F 2 "" H 2300 3700 50  0001 C CNN
@@
 $EndComp
 $Comp
-L GND #PWR022
+L GND #PWR020
 U 1 1 5F3C947F
 P 6350 3700
-F 0 "#PWR022" H 6350 3450 50  0001 C CNN
+F 0 "#PWR020" H 6350 3450 50  0001 C CNN
 F 1 "GND" H 6350 3550 50  0000 C CNN
 F 2 "" H 6350 3700 50  0001 C CNN
@@
 	2300 3900 2400 3900
 $Comp
-L +6V #PWR023
+L +6V #PWR021
 U 1 1 5F3C949C
 P 3850 3600
-F 0 "#PWR023" H 3850 3450 50  0001 C CNN
+F 0 "#PWR021" H 3850 3450 50  0001 C CNN
 F 1 "+6V" H 3850 3740 50  0000 C CNN
 F 2 "" H 3850 3600 50  0001 C CNN
@@
 $EndComp
 Wire Wire Line
-	3850 3600 3850 3800
-Wire Wire Line
 	3850 3800 3700 3800
 $Comp
-L +6V #PWR024
+L +6V #PWR022
 U 1 1 5F3C94BD
 P 4700 3550
-F 0 "#PWR024" H 4700 3400 50  0001 C CNN
+F 0 "#PWR022" H 4700 3400 50  0001 C CNN
 F 1 "+6V" H 4700 3690 50  0000 C CNN
 F 2 "" H 4700 3550 50  0001 C CNN
@@
 $EndComp
 Wire Wire Line
-	4700 3550 4700 3800
-Wire Wire Line
 	4700 3800 4900 3800
 $Comp
-L +6V #PWR025
+L +6V #PWR023
 U 1 1 5F3C94D8
 P 3850 4150
-F 0 "#PWR025" H 3850 4000 50  0001 C CNN
+F 0 "#PWR023" H 3850 4000 50  0001 C CNN
 F 1 "+6V" H 3850 4290 50  0000 C CNN
 F 2 "" H 3850 4150 50  0001 C CNN
@@
 $EndComp
 Wire Wire Line
-	3850 4150 3850 4000
-Wire Wire Line
 	3850 4000 3700 4000
 $Comp
-L +6V #PWR026
+L +6V #PWR024
 U 1 1 5F3C94F6
 P 4700 4150
-F 0 "#PWR026" H 4700 4000 50  0001 C CNN
+F 0 "#PWR024" H 4700 4000 50  0001 C CNN
 F 1 "+6V" H 4700 4290 50  0000 C CNN
 F 2 "" H 4700 4150 50  0001 C CNN
@@
 	-1   0    0    1
 $EndComp
-Wire Wire Line
-	4700 4150 4700 4000
 Wire Wire Line
 	4700 4000 4900 4000
@@
 F 0 "K1" H 4850 4300 50  0000 L CNN
 F 1 "JQ1P-5V-F" H 4850 4200 50  0000 L CNN
-F 2 "JQ1P5VF" H 4850 4100 50  0001 L CNN
+F 2 "lib:JQ1P5VF" H 4850 4100 50  0001 L CNN
 F 3 "https://www3.panasonic.biz/ac/e_download/control/relay/power/catalog/mech_eng_jq.pdf?via=ok" H 4850 4000 50  0001 L CNN
 F 4 "Electromechanical Relay 5VDC 62.5Ohm 10(NO)/3(NC)A SPDT (20x10x16)mm THT Power Relay" H 4850 3900 50  0001 L CNN "Description"
@@
 	-1   0    0    1
 $EndComp
+Wire Wire Line
+	4700 3800 4700 3550
+Wire Wire Line
+	4700 4000 4700 4150
+Wire Wire Line
+	3850 4000 3850 4150
+Wire Wire Line
+	3850 3600 3850 3800
 $EndSCHEMATC
