File: pcb/power.sch (KiCad schematic (older format))
At the start: 6 parts, among them U4 LD1085D2T33R

Commit message: First submitted PCB
Connections:
- net +BATT renamed ACC_BAT
Changed lines of the file:
@@
 LIBS:PAM8403DR
 LIBS:JQ1P-5V-F
+LIBS:Connector_Generic_MountingPin
 LIBS:controller-cache
 EELAYER 25 0
@@
 Connection ~ 5350 2400
 $Comp
-L +BATT #PWR027
-U 1 1 5F39F126
-P 2850 2400
-F 0 "#PWR027" H 2850 2250 50  0001 C CNN
-F 1 "+BATT" H 2850 2540 50  0000 C CNN
-F 2 "" H 2850 2400 50  0001 C CNN
-F 3 "" H 2850 2400 50  0001 C CNN
-	1    2850 2400
-	0    -1   -1   0
-$EndComp
-$Comp
-L +3V3 #PWR028
+L +3V3 #PWR025
 U 1 1 5F39F146
 P 5600 2400
-F 0 "#PWR028" H 5600 2250 50  0001 C CNN
+F 0 "#PWR025" H 5600 2250 50  0001 C CNN
 F 1 "+3V3" H 5600 2540 50  0000 C CNN
 F 2 "" H 5600 2400 50  0001 C CNN
@@
 	0    1    1    0
 $EndComp
-Wire Wire Line
-	3400 2400 4200 2400
 $Comp
 L Fuse F1
@@
 	2850 2400 3100 2400
 $Comp
-L +6V #PWR029
-U 1 1 5F39F34C
-P 3600 2400
-F 0 "#PWR029" H 3600 2250 50  0001 C CNN
-F 1 "+6V" H 3600 2540 50  0000 C CNN
-F 2 "" H 3600 2400 50  0001 C CNN
-F 3 "" H 3600 2400 50  0001 C CNN
-	1    3600 2400
-	1    0    0    -1
-$EndComp
-$Comp
-L PWR_FLAG #FLG030
-U 1 1 5F3D3CAF
-P 3850 2400
-F 0 "#FLG030" H 3850 2475 50  0001 C CNN
-F 1 "PWR_FLAG" H 3850 2550 50  0000 C CNN
-F 2 "" H 3850 2400 50  0001 C CNN
-F 3 "" H 3850 2400 50  0001 C CNN
-	1    3850 2400
-	1    0    0    -1
-$EndComp
-$Comp
-L PWR_FLAG #FLG031
-U 1 1 5F3D3CCF
-P 3000 2400
-F 0 "#FLG031" H 3000 2475 50  0001 C CNN
-F 1 "PWR_FLAG" H 3000 2550 50  0000 C CNN
-F 2 "" H 3000 2400 50  0001 C CNN
-F 3 "" H 3000 2400 50  0001 C CNN
-	1    3000 2400
-	1    0    0    -1
-$EndComp
-$Comp
-L GND #PWR032
+L GND #PWR026
 U 1 1 5F3D3D27
 P 4800 2700
-F 0 "#PWR032" H 4800 2450 50  0001 C CNN
+F 0 "#PWR026" H 4800 2450 50  0001 C CNN
 F 1 "GND" H 4800 2550 50  0000 C CNN
 F 2 "" H 4800 2700 50  0001 C CNN
@@
 	1    0    0    -1
 $EndComp
-Connection ~ 3000 2400
-Connection ~ 3850 2400
 Connection ~ 4800 2700
 $Comp
-L PWR_FLAG #FLG033
-U 1 1 5F3D5B0F
-P 4200 2700
-F 0 "#FLG033" H 4200 2775 50  0001 C CNN
-F 1 "PWR_FLAG" H 4200 2850 50  0000 C CNN
-F 2 "" H 4200 2700 50  0001 C CNN
-F 3 "" H 4200 2700 50  0001 C CNN
-	1    4200 2700
-	-1   0    0    1
+L +6V #PWR027
+U 1 1 5F3CB177
+P 3600 2300
+F 0 "#PWR027" H 3600 2150 50  0001 C CNN
+F 1 "+6V" H 3600 2440 50  0000 C CNN
+F 2 "" H 3600 2300 50  0001 C CNN
+F 3 "" H 3600 2300 50  0001 C CNN
+	1    3600 2300
+	1    0    0    -1
 $EndComp
-Connection ~ 4200 2700
+Wire Wire Line
+	3600 2300 3600 2400
+Wire Wire Line
+	3400 2400 4200 2400
+Text GLabel 2850 2400 0    60   Input ~ 0
+ACC_BAT
 $EndSCHEMATC
